Commit message: Set rangefinder position

File: rover_sim/urdf/rover_description.urdf (robot description, URDF)
Before this commit: robot rover_description, 26 links, 25 joints
Joints:
- joint scan_joint: origin xyz=-.075 0.03 -.075 rpy=0 -0.275 0 -> xyz=-.075 0.03 -.5125 rpy=0 0 3.14

Commit message: Add new world for obstacle avoidance

File: rover_sim/urdf/rover_description.urdf (robot description, URDF)
Before this commit: robot rover_description, 26 links, 25 joints
Joints:
- joint scan_joint: origin xyz=-.075 0.03 -.5125 rpy=0 0 3.14 -> xyz=-.075 0.03 -.5125 rpy=0.05 0.05 3.14

Commit message: slight errors in avoidance but working

File: rover_sim/urdf/rover_description.urdf (robot description, URDF)
Before this commit: robot rover_description, 26 links, 25 joints
Joints:
- joint scan_joint: origin xyz=-.075 0.03 -.075 rpy=0 -0.275 0 -> xyz=-.075 0.03 -.5125 rpy=0.05 0.05 3.14
